File: Hardware/Modules/7-Segment_Anzeige/7-Segment_MAX7221CNG_.kicad_sch (KiCad schematic)
At the start: 5 parts, among them J2 B6B-EH-A, U1 MAX7221xNG, U4 CC56-12SURKWA, U5 CC56-12SURKWA

Commit message: fixed connector orientation
Parts:
- J2: footprint Connector:CONN_B6B-EH-A_JST -> Connector_JST:JST_EH_B6B-EH-A_1x06_P2.50mm_Vertical
Changed lines of the file:
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@@
 			)
 		)
-		(property "Footprint" "Connector:CONN_B6B-EH-A_JST"
+		(property "Footprint" "Connector_JST:JST_EH_B6B-EH-A_1x06_P2.50mm_Vertical"
 			(at 49.53 99.06 0)
 			(effects

Commit message: fixed GND/VCC issue and added filling zone
Connections:
- net at R2.1, U1.19 (V+): now also J2.1; no longer J2.6
- net at U1.4 (GND), U1.9 (GND): now also J2.6; no longer J2.1
Changed lines of the file:
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@@
+	(wire
+		(pts
+			(xy 49.53 99.06) (xy 63.5 99.06)
+		)
+		(stroke
+			(width 0)
+			(type default)
+		)
+	)
 	(wire
 		(pts
@@
 	(wire
 		(pts
-			(xy 49.53 86.36) (xy 67.31 86.36)
-		)
-		(stroke
-			(width 0)
-			(type default)
-		)
-	)
-	(wire
-		(pts
 			(xy 100.33 118.11) (xy 58.42 118.11)
 		)
@@
 	(wire
 		(pts
-			(xy 58.42 118.11) (xy 58.42 99.06)
+			(xy 58.42 86.36) (xy 58.42 118.11)
 		)
 		(stroke
@@
 	(wire
 		(pts
+			(xy 63.5 86.36) (xy 67.31 86.36)
+		)
+		(stroke
+			(width 0)
+			(type default)
+		)
+	)
+	(wire
+		(pts
 			(xy 205.74 110.49) (xy 203.2 110.49)
 		)
@@
 	(wire
 		(pts
+			(xy 63.5 99.06) (xy 63.5 86.36)
+		)
+		(stroke
+			(width 0)
+			(type default)
+		)
+	)
+	(wire
+		(pts
 			(xy 203.2 83.82) (xy 209.55 83.82)
 		)
@@
 	(wire
 		(pts
-			(xy 58.42 99.06) (xy 49.53 99.06)
-		)
-		(stroke
-			(width 0)
-			(type default)
-		)
-	)
-	(wire
-		(pts
 			(xy 147.32 113.03) (xy 146.05 113.03)
 		)
@@
 		(pts
 			(xy 138.43 120.65) (xy 138.43 102.87)
+		)
+		(stroke
+			(width 0)
+			(type default)
+		)
+	)
+	(wire
+		(pts
+			(xy 58.42 86.36) (xy 49.53 86.36)
 		)
 		(stroke
@@
 	(text "VCC"
 		(exclude_from_sim no)
-		(at 50.546 85.598 0)
+		(at 51.054 98.044 0)
 		(effects
 			(font
@@
 	(text "GND"
 		(exclude_from_sim no)
-		(at 51.054 98.298 0)
+		(at 50.8 85.09 0)
 		(effects
 			(font

Commit message: Added capacitors to 7-segment display
Parts:
- added C1: 10µF, Capacitor_SMD:C_Elec_3x5.4, symbol Device:C
- added C2: 0.1µF, Capacitor_SMD:C_0603_1608Metric_Pad1.08x0.95mm_HandSolder, symbol Device:C
Connections:
- net at J2.1, R2.1, U1.19 (V+): now also C1.1, C2.1
- net at J2.6, U1.4 (GND), U1.9 (GND): now also C1.2, C2.2
Changed lines of the file:
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@@
+	)
+	(junction
+		(at 87.63 63.5)
+		(diameter 0)
+		(color 0 0 0 0)
 	)
 	(junction
@@
 	)
 	(junction
+		(at 73.66 118.11)
+		(diameter 0)
+		(color 0 0 0 0)
+	)
+	(junction
 		(at 67.31 69.85)
+		(diameter 0)
+		(color 0 0 0 0)
+	)
+	(junction
+		(at 87.63 118.11)
 		(diameter 0)
 		(color 0 0 0 0)
@@
 	)
 	(junction
+		(at 73.66 63.5)
+		(diameter 0)
+		(color 0 0 0 0)
+	)
+	(junction
 		(at 144.78 85.09)
 		(diameter 0)
@@
 	(wire
 		(pts
-			(xy 67.31 63.5) (xy 100.33 63.5)
+			(xy 67.31 63.5) (xy 73.66 63.5)
+		)
+		(stroke
+			(width 0)
+			(type default)
+		)
+	)
+	(wire
+		(pts
+			(xy 87.63 91.44) (xy 87.63 118.11)
 		)
 		(stroke
@@
 	(wire
 		(pts
+			(xy 58.42 118.11) (xy 73.66 118.11)
+		)
+		(stroke
+			(width 0)
+			(type default)
+		)
+	)
+	(wire
+		(pts
 			(xy 49.53 93.98) (xy 69.85 93.98)
 		)
@@
 	(wire
 		(pts
+			(xy 73.66 63.5) (xy 87.63 63.5)
+		)
+		(stroke
+			(width 0)
+			(type default)
+		)
+	)
+	(wire
+		(pts
 			(xy 209.55 83.82) (xy 209.55 123.19)
 		)
@@
 	(wire
 		(pts
-			(xy 100.33 118.11) (xy 58.42 118.11)
+			(xy 100.33 118.11) (xy 87.63 118.11)
 		)
 		(stroke
@@
 	(wire
 		(pts
+			(xy 73.66 118.11) (xy 87.63 118.11)
+		)
+		(stroke
+			(width 0)
+			(type default)
+		)
+	)
+	(wire
+		(pts
 			(xy 140.97 118.11) (xy 204.47 118.11)
 		)
@@
 	(wire
 		(pts
+			(xy 73.66 63.5) (xy 73.66 80.01)
+		)
+		(stroke
+			(width 0)
+			(type default)
+		)
+	)
+	(wire
+		(pts
 			(xy 147.32 81.28) (xy 144.78 81.28)
 		)
@@
 	(wire
 		(pts
+			(xy 87.63 63.5) (xy 100.33 63.5)
+		)
+		(stroke
+			(width 0)
+			(type default)
+		)
+	)
+	(wire
+		(pts
 			(xy 139.7 100.33) (xy 139.7 74.93)
 		)
@@
 	(wire
 		(pts
+			(xy 73.66 87.63) (xy 73.66 118.11)
+		)
+		(stroke
+			(width 0)
+			(type default)
+		)
+	)
+	(wire
+		(pts
 			(xy 72.39 120.65) (xy 72.39 91.44)
 		)
@@
 		(pts
 			(xy 58.42 86.36) (xy 49.53 86.36)
+		)
+		(stroke
+			(width 0)
+			(type default)
+		)
+	)
+	(wire
+		(pts
+			(xy 87.63 63.5) (xy 87.63 83.82)
 		)
 		(stroke
@@
 	)
 	(symbol
+		(lib_id "Device:C")
+		(at 87.63 87.63 0)
+		(unit 1)
+		(exclude_from_sim no)
+		(in_bom yes)
+		(on_board yes)
+		(dnp no)
+		(fields_autoplaced yes)
+		(property "Reference" "C1"
+			(at 91.44 86.3599 0)
+			(effects
+				(font
+					(size 1.27 1.27)
+				)
+				(justify left)
+			)
+		)
+		(property "Value" "10µF"
+			(at 91.44 88.8999 0)
+			(effects
+				(font
+					(size 1.27 1.27)
+				)
+				(justify left)
+			)
+		)
+		(property "Footprint" "Capacitor_SMD:C_Elec_3x5.4"
+			(at 88.5952 91.44 0)
+			(effects
+				(font
+					(size 1.27 1.27)
+				)
+				(hide yes)
+			)
+		)
+		(property "Datasheet" "~"
+			(at 87.63 87.63 0)
+			(effects
+				(font
+					(size 1.27 1.27)
+				)
+				(hide yes)
+			)
+		)
+		(property "Description" "Unpolarized capacitor"
+			(at 87.63 87.63 0)
+			(effects
+				(font
+					(size 1.27 1.27)
+				)
+				(hide yes)
+			)
+		)
+		(pin "2"
+		)
+		(pin "1"
+		)
+		(instances
+			(project ""
+				(path "/f950633f-0c21-436d-987a-15b561757a69"
+					(reference "C1")
+					(unit 1)
+				)
+			)
+		)
+	)
+	(symbol
 		(lib_id "Driver_LED:MAX7221xNG")
 		(at 100.33 90.17 0)
@@
 					(unit 1)
 				)
+			)
+		)
+	)
+	(symbol
+		(lib_id "Device:C")
+		(at 73.66 83.82 0)
+		(unit 1)
+		(exclude_from_sim no)
+		(in_bom yes)
+		(on_board yes)
+		(dnp no)
+		(fields_autoplaced yes)
+		(property "Reference" "C2"
+			(at 77.47 82.5499 0)
+			(effects
+				(font
+					(size 1.27 1.27)
+				)
+				(justify left)
+			)
+		)
+		(property "Value" "0.1µF"
+			(at 77.47 85.0899 0)
+			(effects
+				(font
+					(size 1.27 1.27)
+				)
+				(justify left)
+			)
+		)
+		(property "Footprint" "Capacitor_SMD:C_0603_1608Metric_Pad1.08x0.95mm_HandSolder"
+			(at 74.6252 87.63 0)
+			(effects
+				(font
+					(size 1.27 1.27)
+				)
+				(hide yes)
+			)
+		)
+		(property "Datasheet" "~"
+			(at 73.66 83.82 0)
+			(effects
+				(font
+					(size 1.27 1.27)
+				)
+				(hide yes)
+			)
+		)
+		(property "Description" "Unpolarized capacitor"
+			(at 73.66 83.82 0)
+			(effects
+				(font
+					(size 1.27 1.27)
+				)
+				(hide yes)
+			)
+		)
+		(pin "2"
+		)
+		(pin "1"
+		)
+		(instances
+			(project "7-Segment_MAX7221CNG_"
+				(path "/f950633f-0c21-436d-987a-15b561757a69"
+					(reference "C2")
+					(unit 1)
+				)
