File: Hardware/Modules/Flight-Module/Flight-module.kicad_pcb (KiCad board)
At the start: 2 copper layers, 35 x 35 mm, 31 parts, among them J3 Conn_01x01_Pin, J4 B6B-EH-A, J5 B6B-EH-A, J6 Conn_01x01_Pin, J7 Conn_01x01_Pin, U1 BMP390, U2 SAM-M10Q-00B, U3 PCA9306DCTR, U4 ICM-20948, U5 TLV70018_SOT23-5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

Commit message: Finishing Modules
Wifi-Module
Flight-Module
REPAIR:
- Heartrate
- Flight-Module
- Wifi-Module
Connections:
- U5 pad 3: unconnected-(U5-EN-Pad3) -> VCC
- U6 pad 3: unconnected-(U6-EN-Pad3) -> VCC
Routing:
- net VCC: track 79.4 -> 88.2 mm, vias 3 -> 6

Commit message: Pushing Final Versions of all Modules (2025)
Parts:
- U1: footprint Modular_Electronics_Toolkit_Footprints:10LGA_2X2X0p75_BOS -> Modular-Elektronics-Toolkit-Global-Libary:10LGA_2X2X0p75_BOS
- U2: footprint Modular_Electronics_Toolkit_Footprints:XCVR_SAM-M10Q-00B -> Modular-Elektronics-Toolkit-Global-Libary:XCVR_SAM-M10Q-00B
- U3, U7, U8: footprint Modular_Electronics_Toolkit_Footprints:SOP65P400X130-8N -> Modular-Elektronics-Toolkit-Global-Libary:SOP65P400X130-8N
